File: AvionicsGPSModule.kicad_pcb (KiCad board)
At the start: 4 copper layers, 60 x 56.1 mm, 32 parts, among them P1 MC311D, Q1 AO3400A, U1 RP2040, U2 AP2112K-3.3, U3 L80-R, U4 W25Q128JVS, X1 ABM8-272-T3

Commit message: finalized wiring
Parts:
- R3: value 200 -> 330
Routing:
- net +5V: track 7.89 -> 41.7 mm
- net /XIN: track 5.39 -> 9.67 mm
- net /QSPI_SS: track 18.3 -> 19.9 mm
- net GND: track 16.9 -> 17.3 mm, vias 25 -> 26
